File: hardware/CPU.kicad_sch (KiCad schematic)
At the start: 43 parts, among them J2 2032 battery, J3 DF4-20DP-2C, J4 DF4-20DP-2C, J6 POWER INPUT, J7 1WIRE, J8 SPEAKER, J9 BME280, SW1 Button 1, SW2 Button 2, SW3 Button 3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

Commit message: Update
Parts:
- removed J3, J4: DF4-20DP-2C, 8080clock_w:PinHeader_2x10_P2.54mm_Vertical, symbol 8088clock_w:DF4-20DP-2C
- removed JP1, JP2: Jumper_3_Open, 8080clock:PinHeader_1x03_P2.54mm_Vertical, symbol 8088clock_w:Jumper_3_Open
- removed R19, R20: 0, 8080clock:R_Axial_DIN0207_L6.3mm_D2.5mm_P10.16mm_Horizontal, symbol 8088clock_w:R
- added C29: 10u, 8080clock:CP_Radial_D5.0mm_P2.50mm, symbol 8088clock_w:C_Polarized
- added C30: 0.1u, 8080clock:C_Disc_D7.0mm_W2.5mm_P5.00mm, symbol 8088clock_w:C
- added C31: 0.1uF, 8080clock_w:C_Disc_D7.0mm_W2.5mm_P5.00mm, symbol 8088clock_w:C
Connections:
- net +5MAIN: now also U8.1 (VPP), C29.1, C30.2, C31.2
- net 1WIRE: now also RN1.2 (R1); no longer RN1.3 (R2)
- net A12: now also U7.2 (A12), U8.2 (A12); no longer U7.1 (A14)
- net A14: now also U7.1 (A14), U8.27 (A14); no longer U7.2 (A12), U8.2 (A12)
- net BTN1: now also RN1.5 (R4); no longer RN1.6 (R5)
- net BTN2: now also RN1.4 (R3); no longer RN1.5 (R4)
- net BTN3: now also RN1.3 (R2); no longer RN1.4 (R3)
- net GND: now also C29.2, C30.1, C31.1
- net SCL: now also RN1.7 (R6); no longer RN1.8 (R7)
- net SDA: now also RN1.6 (R5); no longer RN1.7 (R6)
Other:
- note removed: "-"
- note removed: "J3"
- note removed: "J4"
- note removed: "R19"
- note removed: "R20"
- moved on the sheet: SW1, SW2, SW3

Commit message: Update
Parts:
- SCR1: value ~ -> (none)
