File: hardware/power.kicad_sch (KiCad schematic)
At the start: 52 parts, among them J1 4840-2201, J10 POWER OUTPUT, Q1 IRF4905, Q2 IRF4905, Q3 КТ361В, U1 NE555N, U2 L7905ACV, U3 TPS54260

Commit message: Update
Parts:
- removed Q3: КТ361В, 8080clock:КТ361В, symbol 8088clock_w:КТ315
- added Q3: BC547, Package_TO_SOT_THT:TO-92L_Inline, symbol Transistor_BJT:BC547
Connections:
- net GND: now also Q3.3 (E)
- net at R6.2, R8.1: now also Q3.2 (B)
- net at R10.1, R13.1: now also Q3.1 (C)
Changed lines of the file:
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@@
 	(wire
 		(pts
-			(xy 224.79 264.16) (xy 228.6 264.16)
+			(xy 224.79 264.16) (xy 229.87 264.16)
 		)
 		(stroke
@@
 	(wire
 		(pts
+			(xy 237.49 252.73) (xy 237.49 259.08)
+		)
+		(stroke
+			(width 0)
+			(type default)
+		)
+	)
+	(wire
+		(pts
 			(xy 224.79 238.76) (xy 224.79 241.3)
 		)
@@
 	(wire
 		(pts
-			(xy 237.49 252.73) (xy 237.49 257.81)
-		)
-		(stroke
-			(width 0)
-			(type default)
-		)
-	)
-	(wire
-		(pts
 			(xy 204.47 96.52) (xy 204.47 91.44)
 		)
@@
 	(wire
 		(pts
-			(xy 237.49 270.51) (xy 237.49 274.32)
+			(xy 237.49 269.24) (xy 237.49 274.32)
 		)
 		(stroke
@@
 	)
 	(symbol
-		(lib_id "8088clock_w:КТ315")
-		(at 234.95 264.16 0)
-		(unit 1)
-		(exclude_from_sim no)
-		(in_bom yes)
-		(on_board yes)
-		(dnp no)
-		(property "Reference" "Q3"
-			(at 232.918 259.842 0)
-			(effects
-				(font
-					(size 1.27 1.27)
-				)
-			)
-		)
-		(property "Value" "КТ361В"
-			(at 231.14 268.478 0)
-			(effects
-				(font
-					(size 1.27 1.27)
-				)
-			)
-		)
-		(property "Footprint" "8080clock:КТ361В"
-			(at 234.95 264.16 0)
-			(effects
-				(font
-					(size 1.27 1.27)
-				)
-				(hide yes)
-			)
-		)
-		(property "Datasheet" ""
-			(at 234.95 264.16 0)
-			(effects
-				(font
-					(size 1.27 1.27)
-				)
-				(hide yes)
-			)
-		)
-		(property "Description" "PNP Transistor, KT-13"
-			(at 234.95 264.16 0)
-			(effects
-				(font
-					(size 1.27 1.27)
-				)
-				(hide yes)
-			)
-		)
-		(property "Sim.Pins" ""
-			(at 234.95 264.16 0)
-			(effects
-				(font
-					(size 1.27 1.27)
-				)
-				(hide yes)
-			)
-		)
-		(pin "2"
-		)
-		(pin "1"
-		)
-		(pin "3"
-		)
-		(instances
-			(project "8080clock"
-				(path "/acb78ea8-ed4c-41a7-9153-6783241a9453/f94da994-97d5-4817-89a5-9f11c4c7d7d9"
-					(reference "Q3")
-					(unit 1)
-				)
-			)
-		)
-	)
-	(symbol
 		(lib_id "8088clock_w:LED")
 		(at 318.77 90.17 270)
@@
 					(unit 1)
 				)
+			)
+		)
+	)
+	(symbol
+		(lib_id "Transistor_BJT:BC547")
+		(at 234.95 264.16 0)
+		(unit 1)
+		(exclude_from_sim no)
+		(in_bom yes)
+		(on_board yes)
+		(dnp no)
+		(fields_autoplaced yes)
+		(property "Reference" "Q3"
+			(at 240.03 262.8899 0)
+			(effects
+				(font
+					(size 1.27 1.27)
+				)
+				(justify left)
+			)
+		)
+		(property "Value" "BC547"
+			(at 240.03 265.4299 0)
+			(effects
+				(font
+					(size 1.27 1.27)
+				)
+				(justify left)
+			)
+		)
+		(property "Footprint" "Package_TO_SOT_THT:TO-92L_Inline"
+			(at 240.03 266.065 0)
+			(effects
+				(font
+					(size 1.27 1.27)
+					(italic yes)
+				)
+				(justify left)
+				(hide yes)
+			)
+		)
+		(property "Datasheet" "https://www.onsemi.com/pub/Collateral/BC550-D.pdf"
+			(at 234.95 264.16 0)
+			(effects
+				(font
+					(size 1.27 1.27)
+				)
+				(justify left)
+				(hide yes)
+			)
+		)
+		(property "Description" "0.1A Ic, 45V Vce, Small Signal NPN Transistor, TO-92"
+			(at 234.95 264.16 0)
+			(effects
+				(font
+					(size 1.27 1.27)
+				)
+				(hide yes)
+			)
+		)
+		(property "Sim.Device" "NPN"
+			(at 234.95 264.16 0)
+			(effects
+				(font
+					(size 1.27 1.27)
+				)
+				(hide yes)
+			)
+		)
+		(property "Sim.Pins" "1=C 2=B 3=E"
+			(at 234.95 264.16 0)
+			(effects
+				(font
+					(size 1.27 1.27)
+				)
+				(hide yes)
+			)
+		)
+		(pin "1"
+		)
+		(pin "3"
+		)
+		(pin "2"
+		)
+		(instances
+			(project ""
+				(path "/acb78ea8-ed4c-41a7-9153-6783241a9453/f94da994-97d5-4817-89a5-9f11c4c7d7d9"
+					(reference "Q3")
+					(unit 1)
+				)

Commit message: Update
Parts:
- Q3: value BC547 -> BC337
