File: hardware/8080clock.kicad_pcb (KiCad board)
At the start: 2 copper layers, 199.7 x 119.9 mm, 105 parts, among them J1 4840-2201, J10 POWER OUTPUT, J2 2032 battery, J6 POWER INPUT, J7 1WIRE, J8 SPEAKER, J9 BME280, M1 MountingHole_2.7mm_M2.5, M2 MountingHole_2.7mm_M2.5, M3 MountingHole_2.7mm_M2.5, M4 MountingHole_2.7mm_M2.5, M5 MountingHole_2.7mm_M2.5, M6 MountingHole_2.7mm_M2.5, M7 MountingHole_2.7mm_M2.5, M8 MountingHole_2.7mm_M2.5, Q1 IRF4905, Q2 IRF4905, Q3 КТ361В, SW1 Button 1, SW2 Button 2, SW3 Button 3, SW4 RESET, U1 NE555N, U10 Intel 8255A / КР580ВВ55А, U11 PCF8563P, U12 Intel 8080 / КР580ВМ80, U2 L7905ACV, U3 TPS54260, U5 Intel 8224 / КР580ГФ24, U6 Intel 8238 / КР580ВК38, U7 CY62256L-70PC, U8 27C256 / КР573РФ8, U9 74LS04 / К555ЛН1, Y1 32MHZ, Y2 32.768

Commit message: Gerbers
Other:
- board text added: "Based on i8080 clock by Tronix286 github.com/Tronix286/i8080_clock"
- board text added: "Double PCB version by MadCat, 2025-2026 github.com/madcatse/8080_desktop_clock t.me/madcatse Version 0.1"
- board text removed: "Based on i8080 clock by Tronix286 github.com/Tronix286/i8080_clock Double PCB version by MadCat, 2025-2026 github.com/madcatse/8080_desktop_clock t.me/madcatse Version 0.1"
Changed lines of the file:
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@@
 			(outputformat 1)
 			(mirror no)
-			(drillshape 1)
+			(drillshape 0)
 			(scaleselection 1)
-			(outputdirectory "")
+			(outputdirectory "gerber/")
 		)
 	)
@@
 		)
 	)
-	(gr_text "Based on i8080 clock\nby Tronix286\ngithub.com/Tronix286/i8080_clock\n\nDouble PCB version \nby MadCat, 2025-2026\ngithub.com/madcatse/8080_desktop_clock\nt.me/madcatse\nVersion 0.1"
-		(at 203.2508 75.7428 180)
+	(gr_text "Double PCB version \nby MadCat, 2025-2026\ngithub.com/madcatse/8080_desktop_clock\nt.me/madcatse\nVersion 0.1"
+		(at 202.5396 78.4352 180)
 		(layer "F.SilkS")
 		(effects
@@
 		)
 	)
+	(gr_text "Based on i8080 clock\nby Tronix286\ngithub.com/Tronix286/i8080_clock"
+		(at 201.5236 90.678 180)
+		(layer "F.SilkS")
+		(effects
+			(font
+				(size 1 1)
+				(thickness 0.15)
+			)
+		)
+	)

Commit message: Small fixes for holes
Parts:
- M1, M2, M3, M4, M5, M6, M7, M8: value MountingHole_2.7mm_M2.5 -> MountingHole_3.2mm_M3.0; footprint 8080clock:MountingHole_2.7mm_M2.5 -> 8080clock:MountingHole_3.2mm_M3.0
Changed lines of the file:
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@@
 		)
 	)
-	(footprint "8080clock:MountingHole_2.7mm_M2.5"
+	(footprint "8080clock:MountingHole_3.2mm_M3.0"
 		(layer "F.Cu")
 		(at 269.348 71.564)
@@
 			)
 		)
-		(property "Value" "MountingHole_2.7mm_M2.5"
+		(property "Value" "MountingHole_3.2mm_M3.0"
 			(at 0 3.65 0)
 			(layer "F.Fab")
@@
 		(pad "" np_thru_hole circle
 			(at 0 0)
-			(size 2.7 2.7)
-			(drill 2.7)
+			(size 3.2 3.2)
+			(drill 3.2)
 			(layers "*.Cu" "*.Mask")
 		)
@@
 		(embedded_fonts no)
 	)
-	(footprint "8080clock:MountingHole_2.7mm_M2.5"
+	(footprint "8080clock:MountingHole_3.2mm_M3.0"
 		(layer "F.Cu")
 		(at 269.348 183.452)
@@
 			)
 		)
-		(property "Value" "MountingHole_2.7mm_M2.5"
+		(property "Value" "MountingHole_3.2mm_M3.0"
 			(at 0 3.65 0)
 			(layer "F.Fab")
@@
 		(pad "" np_thru_hole circle
 			(at 0 0)
-			(size 2.7 2.7)
-			(drill 2.7)
+			(size 3.2 3.2)
+			(drill 3.2)
 			(layers "*.Cu" "*.Mask")
 		)
 		(embedded_fonts no)
 	)
-	(footprint "8080clock:MountingHole_2.7mm_M2.5"
+	(footprint "8080clock:MountingHole_3.2mm_M3.0"
 		(layer "F.Cu")
 		(at 269.348 133.008)
@@
 			)
 		)
-		(property "Value" "MountingHole_2.7mm_M2.5"
+		(property "Value" "MountingHole_3.2mm_M3.0"
 			(at 0 3.65 0)
 			(layer "F.Fab")
@@
 		(pad "" np_thru_hole circle
 			(at 0 0)
-			(size 2.7 2.7)
-			(drill 2.7)
+			(size 3.2 3.2)
+			(drill 3.2)
 			(layers "*.Cu" "*.Mask")
 		)
@@
 		(embedded_fonts no)
 	)
-	(footprint "8080clock:MountingHole_2.7mm_M2.5"
+	(footprint "8080clock:MountingHole_3.2mm_M3.0"
 		(layer "F.Cu")
 		(at 77.616 133.008)
@@
 			)
 		)
-		(property "Value" "MountingHole_2.7mm_M2.5"
+		(property "Value" "MountingHole_3.2mm_M3.0"
 			(at 0 3.65 0)
 			(layer "F.Fab")
@@
 		(pad "" np_thru_hole circle
 			(at 0 0)
-			(size 2.7 2.7)
-			(drill 2.7)
+			(size 3.2 3.2)
+			(drill 3.2)
 			(layers "*.Cu" "*.Mask")
 		)
@@
 		)
 	)
-	(footprint "8080clock:MountingHole_2.7mm_M2.5"
+	(footprint "8080clock:MountingHole_3.2mm_M3.0"
 		(layer "F.Cu")
 		(at 77.616 71.564)
@@
 		(tags "mountinghole M2.5")
 		(property "Reference" "M7"
-			(at 4.4768 -0.7488 0)
+			(at 0 -3.65 0)
 			(layer "F.SilkS")
 			(hide yes)
@@
 			)
 		)
-		(property "Value" "MountingHole_2.7mm_M2.5"
+		(property "Value" "MountingHole_3.2mm_M3.0"
 			(at 0 3.65 0)
 			(layer "F.Fab")
@@
 		(pad "" np_thru_hole circle
 			(at 0 0)
-			(size 2.7 2.7)
-			(drill 2.7)
+			(size 3.2 3.2)
+			(drill 3.2)
 			(layers "*.Cu" "*.Mask")
 		)
@@
 		(embedded_fonts no)
 	)
-	(footprint "8080clock:MountingHole_2.7mm_M2.5"
+	(footprint "8080clock:MountingHole_3.2mm_M3.0"
 		(layer "F.Cu")
 		(at 77.616 122.008)
@@
 			)
 		)
-		(property "Value" "MountingHole_2.7mm_M2.5"
+		(property "Value" "MountingHole_3.2mm_M3.0"
 			(at 0 3.65 0)
 			(layer "F.Fab")
@@
 		(pad "" np_thru_hole circle
 			(at 0 0)
-			(size 2.7 2.7)
-			(drill 2.7)
+			(size 3.2 3.2)
+			(drill 3.2)
 			(layers "*.Cu" "*.Mask")
 		)
@@
 		(embedded_fonts no)
 	)
-	(footprint "8080clock:MountingHole_2.7mm_M2.5"
+	(footprint "8080clock:MountingHole_3.2mm_M3.0"
 		(layer "F.Cu")
 		(at 77.616 183.452)
@@
 			)
 		)
-		(property "Value" "MountingHole_2.7mm_M2.5"
+		(property "Value" "MountingHole_3.2mm_M3.0"
 			(at 0 3.65 0)
 			(layer "F.Fab")
@@
 		(pad "" np_thru_hole circle
 			(at 0 0)
-			(size 2.7 2.7)
-			(drill 2.7)
+			(size 3.2 3.2)
+			(drill 3.2)
 			(layers "*.Cu" "*.Mask")
 		)
@@
 		)
 	)
-	(footprint "8080clock:MountingHole_2.7mm_M2.5"
+	(footprint "8080clock:MountingHole_3.2mm_M3.0"
 		(layer "F.Cu")
 		(at 269.348 122.008)
@@
 			)
 		)
-		(property "Value" "MountingHole_2.7mm_M2.5"
+		(property "Value" "MountingHole_3.2mm_M3.0"
 			(at 0 3.65 0)
 			(layer "F.Fab")
@@
 		(pad "" np_thru_hole circle
 			(at 0 0)
-			(size 2.7 2.7)
-			(drill 2.7)
+			(size 3.2 3.2)
+			(drill 3.2)
 			(layers "*.Cu" "*.Mask")
 		)

Commit message: Update
Parts:
- removed JP1, JP2: Jumper_3_Open, 8080clock:PinHeader_1x03_P2.54mm_Vertical
- removed R19, R20: 0, 8080clock:R_Axial_DIN0207_L6.3mm_D2.5mm_P10.16mm_Horizontal
- added C22: 0.1uF, 8080clock_w:C_Disc_D7.0mm_W2.5mm_P5.00mm, B.Cu at (250.2, 98.0)
- added C29: 10u, 8080clock:CP_Radial_D5.0mm_P2.50mm, B.Cu at (241.6, 76.9)
- added C30: 0.1u, 8080clock:C_Disc_D7.0mm_W2.5mm_P5.00mm, B.Cu at (237.8, 72.5)
- added C31: 0.1uF, 8080clock_w:C_Disc_D7.0mm_W2.5mm_P5.00mm, B.Cu at (228.0, 109.7)
- Q3: value КТ361В -> BC547; footprint 8080clock:КТ361В -> Package_TO_SOT_THT:TO-92L_Inline
- moved mouse-bite-2.54mm-slot_13 192.6 mm to (269.7, 124.5), turned to 180 degrees
- moved mouse-bite-2.54mm-slot_7 192.6 mm to (77.2, 124.5), turned to 180 degrees
- moved mouse-bite-2.54mm-slot_1 137.6 mm to (242.2, 124.5), turned to 180 degrees
- moved mouse-bite-2.54mm-slot_6 137.6 mm to (104.7, 124.5), turned to 180 degrees
- moved mouse-bite-2.54mm-slot_2 82.6 mm to (214.7, 124.5), turned to 180 degrees
- moved mouse-bite-2.54mm-slot_5 82.6 mm to (132.2, 124.5), turned to 180 degrees
- moved C27 65.6 mm to (198.6, 69.8)
- moved RN1 64.6 mm to (167.1, 85.5)
- moved J7 64.4 mm to (253.5, 85.8)
- moved J8 64.4 mm to (258.1, 85.8)
- moved M3 64.4 mm to (77.6, 68.6)
- moved M4 64.4 mm to (269.3, 68.6)
- moved SCR1 64.4 mm to (247.0, 118.0)
- moved U7 64.4 mm to (224.0, 112.2)
- moved D7 64.4 mm to (188.2, 80.7)
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Connections:
- Q3 pad 1: GND -> Net-(Q3-C)
- Q3 pad 2: Net-(Q3-К) -> Net-(Q3-B)
- Q3 pad 3: Net-(Q3-Б) -> GND
- R10 pad 1: Net-(Q3-К) -> Net-(Q3-C)
- R13 pad 1: Net-(Q3-К) -> Net-(Q3-C)
- R6 pad 2: Net-(Q3-Б) -> Net-(Q3-B)
- R8 pad 1: Net-(Q3-Б) -> Net-(Q3-B)
- RN1 pad 2: unconnected-(RN1-R1-Pad2) -> 1WIRE
- RN1 pad 3: 1WIRE -> BTN3
- RN1 pad 4: BTN3 -> BTN2
- RN1 pad 5: BTN2 -> BTN1
- RN1 pad 6: BTN1 -> SDA
- RN1 pad 7: SDA -> SCL
- RN1 pad 8: SCL -> unconnected-(RN1-R7-Pad8)
- U7 pad 1: /CPU/A12 -> /CPU/A14
- U7 pad 2: /CPU/A14 -> /CPU/A12
- U8 pad 1: Net-(JP2-C) -> +5MAIN
- U8 pad 2: /CPU/A14 -> /CPU/A12
- U8 pad 27: Net-(JP1-C) -> /CPU/A14
Routing:
- net Net-(Q3-C): track 0.00 -> 60.2 mm
- net Net-(Q3-К): track 60.2 -> 0.00 mm
- net Net-(Q3-B): track 0.00 -> 42.3 mm, vias 0 -> 1
- net Net-(Q3-Б): track 41.8 -> 0.00 mm, vias 1 -> 0
- net +5MAIN: track 908.9 -> 944.0 mm, vias 5 -> 6
- net GND: track 2254.3 -> 2282.6 mm, vias 837 -> 9
- net Net-(JP2-C): track 9.87 -> 0.00 mm
- net Net-(U5-XTAL1): track 25.9 -> 16.6 mm
- net Net-(JP1-C): track 6.88 -> 0.00 mm
- net Net-(Y1-OSC2): track 9.70 -> 4.66 mm
- net /CPU/A12: track 168.8 -> 173.8 mm, vias 4 -> 5
- net Net-(U5-XTAL2): track 28.1 -> 23.2 mm
- net BTN2: track 224.7 -> 222.2 mm, vias 4 -> 3
- net /CPU/DB7: track 273.2 -> 271.6 mm
- net /CPU/A0: track 204.9 -> 206.3 mm
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- removed copper zone on B.Cu, net GND
- removed copper zone on F.Cu, net GND
Other:
- board text added: "0.1uF"
- board text added: "Based on i8080 clock by Tronix https://t.me/tronix_blog github.com/Tronix286/i8080_clock Huge thanks for help and support!"
- board text added: "Double PCB version by MadCat, 2025-2026 github.com/madcatse/8080_desktop_clock t.me/madcatse Version 1.0"
- board text removed: "27C256: JP1 1-2 JP2 1-2 27C512: JP1 2-3 JP2 2-3"
- board text removed: "Based on i8080 clock by Tronix286 github.com/Tronix286/i8080_clock"
- board text removed: "Double PCB version by MadCat, 2025-2026 github.com/madcatse/8080_desktop_clock t.me/madcatse Version 0.1"
- board text removed: "JP1: 1-2 GND 2-3 A12 JP2: 1-2 +5V 2-3 A12"

Commit message: Clock Update
Routing:
- net GND: track 2282.6 -> 2281.9 mm

Commit message: Update
Parts:
- Q3: value BC547 -> BC337

Commit message: Update 25.05.2026
Parts:
- moved Y1 1.54 mm to (204.0, 76.5), turned to 0 degrees
Routing:
- net Net-(Y1-OSC2): track 4.66 -> 13.1 mm
- net Net-(U5-XTAL2): track 23.2 -> 22.3 mm, vias 1 -> 0
Changed lines of the file:
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@@
 		(capping no)
 		(filling no)
+		(zone_defaults)
 		(pcbplotparams
 			(layerselection 0x00000000_00000000_55555555_5755f5ff)
@@
 			(drillshape 0)
 			(scaleselection 1)
-			(outputdirectory "gerber/ver1.0/")
+			(outputdirectory "gerber/")
 		)
 	)
@@
 		)
 		(embedded_fonts no)
-		(model "${KICAD9_3DMODEL_DIR}/Connector_PinSocket_2.54mm.3dshapes/PinSocket_1x06_P2.54mm_Vertical.wrl"
+		(model "${KICAD10_3DMODEL_DIR}/Connector_PinSocket_2.54mm.3dshapes/PinSocket_1x06_P2.54mm_Vertical.step"
 			(offset
 				(xyz -29.5 48 0)
@@
 			)
 		)
-		(model "${KICAD9_3DMODEL_DIR}/Connector_PinSocket_2.54mm.3dshapes/PinSocket_1x06_P2.54mm_Vertical.wrl"
+		(model "${KICAD10_3DMODEL_DIR}/Connector_PinSocket_2.54mm.3dshapes/PinSocket_1x06_P2.54mm_Vertical.step"
 			(offset
 				(xyz -11.75 48 0)
@@
 			)
 		)
-		(model "${KICAD9_3DMODEL_DIR}/Connector_PinSocket_2.54mm.3dshapes/PinSocket_1x08_P2.54mm_Vertical.wrl"
+		(model "${KICAD10_3DMODEL_DIR}/Connector_PinSocket_2.54mm.3dshapes/PinSocket_1x08_P2.54mm_Vertical.step"
 			(offset
 				(xyz -29.5 -0.25 0)
@@
 			)
 		)
-		(model "${KICAD9_3DMODEL_DIR}/Connector_PinSocket_2.54mm.3dshapes/PinSocket_1x08_P2.54mm_Vertical.wrl"
+		(model "${KICAD10_3DMODEL_DIR}/Connector_PinSocket_2.54mm.3dshapes/PinSocket_1x08_P2.54mm_Vertical.step"
 			(offset
 				(xyz -7.75 -0.25 0)
@@
 		(tags "C Disc series Radial pin pitch 5.00mm diameter 7mm width 2.5mm Capacitor")
 		(property "Reference" "C30"
-			(at 2.4492 -2.3504 0)
+			(at -2.8348 -0.0128 0)
 			(layer "B.SilkS")
 			(effects
@@
 	(footprint "8080clock:Crystal_HC49-4H_Vertical"
 		(layer "B.Cu")
-		(at 202.946 75.383 90)
+		(at 204 76.5)
 		(descr "HC-49-4H, Crystal, http://5hertz.com/pdfs/04404_D.pdf")
 		(property "Reference" "Y1"
-			(at 9.2456 -0.1524 0)
+			(at 8.5 -3 180)
 			(layer "B.SilkS")
 			(effects
@@
 		)
 		(property "Value" "32MHZ"
-			(at -4.6228 2.54 0)
+			(at 2.4 -3.7 180)
 			(layer "B.SilkS")
 			(effects
@@
 		)
 		(property "Datasheet" ""
-			(at 0 0 90)
+			(at 0 0 0)
 			(layer "B.Fab")
 			(hide yes)
@@
 		)
 		(property "Description" ""
-			(at 0 0 90)
+			(at 0 0 0)
 			(layer "B.Fab")
 			(hide yes)
@@
 		)
 		(property "Sim.Pins" ""
-			(at 0 0 90)
+			(at 0 0 0)
 			(unlocked yes)
 			(layer "B.Fab")
@@
 		(duplicate_pad_numbers_are_jumpers no)
 		(fp_line
-			(start 5.64 -2.435)
-			(end -0.76 -2.435)
-			(stroke
-				(width 0.12)
-				(type solid)
-			)
-			(layer "B.SilkS")
-		)
-		(fp_line
 			(start -0.76 2.435)
 			(end 5.64 2.435)
@@
 			(layer "B.SilkS")
 		)
-		(fp_arc
+		(fp_line
 			(start 5.64 -2.435)
-			(mid 8.075 0)
-			(end 5.64 2.435)
+			(end -0.76 -2.435)
 			(stroke
 				(width 0.12)
@@
 			(layer "B.SilkS")
 		)
-		(fp_line
-			(start 5.64 -2.83)
-			(end -0.76 -2.83)
+		(fp_arc
+			(start 5.64 -2.435)
+			(mid 8.075 0)
+			(end 5.64 2.435)
 			(stroke
-				(width 0.05)
+				(width 0.12)
 				(type solid)
 			)
-			(layer "B.CrtYd")
+			(layer "B.SilkS")
 		)
 		(fp_line
@@
 			(layer "B.CrtYd")
 		)
-		(fp_arc
+		(fp_line
 			(start 5.64 -2.83)
-			(mid 8.47 0)
-			(end 5.64 2.83)
+			(end -0.76 -2.83)
 			(stroke
 				(width 0.05)
@@
 			(layer "B.CrtYd")
 		)
-		(fp_line
-			(start 5.64 -2.325)
-			(end -0.76 -2.325)
+		(fp_arc
+			(start 5.64 -2.83)
+			(mid 8.47 0)
+			(end 5.64 2.83)
 			(stroke
-				(width 0.1)
+				(width 0.05)
 				(type solid)
 			)
-			(layer "B.Fab")
+			(layer "B.CrtYd")
 		)
 		(fp_line
@@
 			(layer "B.Fab")
 		)
-		(fp_arc
+		(fp_line
 			(start 5.64 -2.325)
-			(mid 7.965 0)
-			(end 5.64 2.325)
+			(end -0.76 -2.325)
 			(stroke
 				(width 0.1)
@@
 			(layer "B.Fab")
 		)
+		(fp_arc
+			(start 5.64 -2.325)
+			(mid 7.965 0)
+			(end 5.64 2.325)
+			(stroke
+				(width 0.1)
+				(type solid)
+			)
+			(layer "B.Fab")
+		)
 		(fp_text user "${REFERENCE}"
-			(at 2.44 0 90)
+			(at 2.44 0 0)
 			(layer "B.Fab")
 			(effects
@@
 		)
 		(pad "1" thru_hole circle
-			(at 0 0 90)
+			(at 0 0)
 			(size 1.5 1.5)
 			(drill 0.8)
@@
 		)
 		(pad "2" thru_hole circle
-			(at 4.88 0 90)
+			(at 4.88 0)
 			(size 1.5 1.5)
 			(drill 0.8)
@@
 	(segment
 		(start 182.654 78.795)
-		(end 202.074 78.795)
+		(end 201.705 78.795)
 		(width 0.25)
 		(layer "F.Cu")
@@
 	)
 	(segment
-		(start 182.626 78.767)
-		(end 182.654 78.795)
+		(start 201.705 78.795)
+		(end 204 76.5)
 		(width 0.25)
 		(layer "F.Cu")
@@
 	)
 	(segment
-		(start 202.074 78.795)
-		(end 202.946 77.923)
+		(start 182.626 78.767)
+		(end 182.654 78.795)
 		(width 0.25)
 		(layer "F.Cu")
 		(net "Net-(U5-XTAL2)")
 	)
-	(via
-		(at 202.946 77.923)
-		(size 0.6)
-		(drill 0.3)
-		(layers "F.Cu" "B.Cu")
-		(capping no)
-		(covering
-			(front no)
-			(back no)
-		)
-		(plugging
-			(front no)
-			(back no)
-		)
-		(filling no)
-		(net "Net-(U5-XTAL2)")
-	)
-	(segment
-		(start 202.946 77.923)
-		(end 202.946 75.383)
-		(width 0.25)
-		(layer "B.Cu")
-		(net "Net-(U5-XTAL2)")
-	)
 	(segment
 		(start 182.761 76.092)
@@
 	)
 	(segment
-		(start 202.946 70.503)
-		(end 199.2814 70.503)
+		(start 202.1788 69.7988)
+		(end 208.88 76.5)
 		(width 0.25)
-		(layer "F.Cu")
+		(layer "B.Cu")
 		(net "Net-(Y1-OSC2)")
 	)
 	(segment
-		(start 199.2814 70.503)
-		(end 198.5772 69.7988)
+		(start 198.5772 69.7988)
+		(end 202.1788 69.7988)
 		(width 0.25)
-		(layer "F.Cu")
+		(layer "B.Cu")
 		(net "Net-(Y1-OSC2)")
 	)
